File: pcb/esp32-ac-board/esp32-ac-board.kicad_pcb (KiCad board)
At the start: 2 copper layers, 81.9 x 52.6 mm, 16 parts, among them J1 Conn_01x15, J2 Conn_01x15, J3 Screw_Terminal_01x02, Q1 Q_NPN_BCE, SW1 SW_Push

Commit message: fix button holes
Parts:
- SW1: footprint Button_Switch_THT:SW_PUSH-12mm -> Button_Switch_THT:SW_PUSH-12mm_Wuerth-430476085716
Routing:
- net /BTN: track 95.3 -> 93.3 mm
Changed lines of the file:
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@@
-(kicad_pcb (version 20171130) (host pcbnew "(5.1.2)-1")
+(kicad_pcb (version 20171130) (host pcbnew 5.0.2)
   (general
     (thickness 1.6)
@@
   (page A4)
   (layers
-    (0 F.Cu signal hide)
+    (0 F.Cu signal)
     (31 B.Cu signal hide)
     (32 B.Adhes user hide)
@@
     (zone_45_only no)
     (trace_min 0.2)
+    (segment_width 0.2)
+    (edge_width 0.05)
     (via_size 0.8)
     (via_drill 0.4)
@@
     (uvia_min_size 0.2)
     (uvia_min_drill 0.1)
-    (edge_width 0.05)
-    (segment_width 0.2)
     (pcb_text_width 0.3)
     (pcb_text_size 1.5 1.5)
@@
     )
   )
-  (module Button_Switch_THT:SW_PUSH-12mm (layer F.Cu)
-    (at 132.588 79.756)
-    (descr "SW PUSH 12mm https://www.e-switch.com/system/asset/product_line/data_sheet/143/TL1100.pdf")
-    (tags "tact sw push 12mm")
-    (fp_text reference SW1 (at 6.08 -4.66) (layer F.SilkS)
-      (effects (font (size 1 1) (thickness 0.15)))
-    )
-    (fp_text value SW_Push (at 6.62 9.93) (layer F.Fab)
-      (effects (font (size 1 1) (thickness 0.15)))
-    )
-    (fp_line (start 0.25 8.5) (end 12.25 8.5) (layer F.Fab) (width 0.1))
-    (fp_line (start 0.25 -3.5) (end 12.25 -3.5) (layer F.Fab) (width 0.1))
-    (fp_line (start 12.25 -3.5) (end 12.25 8.5) (layer F.Fab) (width 0.1))
-    (fp_text user %R (at 6.35 2.54) (layer F.Fab)
-      (effects (font (size 1 1) (thickness 0.15)))
-    )
-    (fp_line (start 0.1 -3.65) (end 12.4 -3.65) (layer F.SilkS) (width 0.12))
-    (fp_line (start 12.4 0.93) (end 12.4 4.07) (layer F.SilkS) (width 0.12))
-    (fp_line (start 12.4 8.65) (end 0.1 8.65) (layer F.SilkS) (width 0.12))
-    (fp_line (start 0.1 -0.93) (end 0.1 -3.65) (layer F.SilkS) (width 0.12))
-    (fp_line (start -1.77 -3.75) (end 14.25 -3.75) (layer F.CrtYd) (width 0.05))
-    (fp_line (start -1.77 -3.75) (end -1.77 8.75) (layer F.CrtYd) (width 0.05))
-    (fp_line (start 14.25 8.75) (end 14.25 -3.75) (layer F.CrtYd) (width 0.05))
-    (fp_line (start 14.25 8.75) (end -1.77 8.75) (layer F.CrtYd) (width 0.05))
-    (fp_circle (center 6.35 2.54) (end 10.16 5.08) (layer F.SilkS) (width 0.12))
-    (fp_line (start 0.25 -3.5) (end 0.25 8.5) (layer F.Fab) (width 0.1))
-    (fp_line (start 0.1 8.65) (end 0.1 5.93) (layer F.SilkS) (width 0.12))
-    (fp_line (start 0.1 4.07) (end 0.1 0.93) (layer F.SilkS) (width 0.12))
-    (fp_line (start 12.4 5.93) (end 12.4 8.65) (layer F.SilkS) (width 0.12))
-    (fp_line (start 12.4 -3.65) (end 12.4 -0.93) (layer F.SilkS) (width 0.12))
-    (pad 1 thru_hole oval (at 12.5 0) (size 3.048 1.7272) (drill 0.8128) (layers *.Cu *.Mask)
-      (net 4 GND))
-    (pad 2 thru_hole oval (at 12.5 5) (size 3.048 1.7272) (drill 0.8128) (layers *.Cu *.Mask)
-      (net 19 /BTN))
-    (pad 1 thru_hole oval (at 0 0) (size 3.048 1.7272) (drill 0.8128) (layers *.Cu *.Mask)
-      (net 4 GND))
-    (pad 2 thru_hole oval (at 0 5) (size 3.048 1.7272) (drill 0.8128) (layers *.Cu *.Mask)
-      (net 19 /BTN))
-    (model ${KISYS3DMOD}/Button_Switch_THT.3dshapes/SW_PUSH-12mm.wrl
-      (at (xyz 0 0 0))
-      (scale (xyz 1 1 1))
-      (rotate (xyz 0 0 0))
-    )
-  )
   (module ESP32:Logo (layer B.Cu)
     (at 137.033 109.982 180)
@@
     )
   )
+  (module Button_Switch_THT:SW_PUSH-12mm_Wuerth-430476085716 (layer F.Cu)
+    (at 132.588 79.756)
+    (descr "SW PUSH 12mm http://katalog.we-online.de/em/datasheet/430476085716.pdf")
+    (tags "tact sw push 12mm")
+    (fp_text reference SW1 (at 6.35 -4.66) (layer F.SilkS)
+      (effects (font (size 1 1) (thickness 0.15)))
+    )
+    (fp_text value SW_Push (at 6.35 9.93) (layer F.Fab)
+      (effects (font (size 1 1) (thickness 0.15)))
+    )
+    (fp_circle (center 6.35 2.54) (end 10.92905 2.54) (layer F.SilkS) (width 0.12))
+    (fp_line (start 0.25 -3.5) (end 0.25 8.5) (layer F.Fab) (width 0.1))
+    (fp_line (start 0.25 8.5) (end 12.25 8.5) (layer F.Fab) (width 0.1))
+    (fp_line (start 12.25 8.5) (end 12.25 -3.5) (layer F.Fab) (width 0.1))
+    (fp_line (start 12.25 -3.5) (end 0.25 -3.5) (layer F.Fab) (width 0.1))
+    (fp_line (start 0.1 -1.53) (end 0.1 -3.65) (layer F.SilkS) (width 0.12))
+    (fp_line (start 0.1 -3.65) (end 12.4 -3.65) (layer F.SilkS) (width 0.12))
+    (fp_line (start 12.4 -3.65) (end 12.4 -1.53) (layer F.SilkS) (width 0.12))
+    (fp_line (start 12.4 1.53) (end 12.4 3.47) (layer F.SilkS) (width 0.12))
+    (fp_line (start 12.4 6.53) (end 12.4 8.65) (layer F.SilkS) (width 0.12))
+    (fp_line (start 12.4 8.65) (end 0.1 8.65) (layer F.SilkS) (width 0.12))
+    (fp_line (start 0.1 8.65) (end 0.1 6.53) (layer F.SilkS) (width 0.12))
+    (fp_line (start 0.1 3.47) (end 0.1 1.53) (layer F.SilkS) (width 0.12))
+    (fp_line (start -1.75 -3.75) (end -1.75 8.75) (layer F.CrtYd) (width 0.05))
+    (fp_line (start -1.75 8.75) (end 14.25 8.75) (layer F.CrtYd) (width 0.05))
+    (fp_line (start 14.25 8.75) (end 14.25 -3.75) (layer F.CrtYd) (width 0.05))
+    (fp_line (start 14.25 -3.75) (end -1.75 -3.75) (layer F.CrtYd) (width 0.05))
+    (fp_text user %R (at 6.35 2.54) (layer F.Fab)
+      (effects (font (size 1 1) (thickness 0.15)))
+    )
+    (pad 1 thru_hole oval (at 12.5 0) (size 3 2.5) (drill 1.2) (layers *.Cu *.Mask)
+      (net 4 GND))
+    (pad 2 thru_hole oval (at 12.5 5) (size 3 2.5) (drill 1.2) (layers *.Cu *.Mask)
+      (net 19 /BTN))
+    (pad 1 thru_hole oval (at 0 0) (size 3 2.5) (drill 1.2) (layers *.Cu *.Mask)
+      (net 4 GND))
+    (pad 2 thru_hole oval (at 0 5) (size 3 2.5) (drill 1.2) (layers *.Cu *.Mask)
+      (net 19 /BTN))
+    (model ${KISYS3DMOD}/Button_Switch_THT.3dshapes/SW_PUSH-12mm_Wuerth-430476085716.wrl
+      (at (xyz 0 0 0))
+      (scale (xyz 1 1 1))
+      (rotate (xyz 0 0 0))
+    )
+  )
   (gr_text GND (at 128.905 79.883) (layer F.SilkS)
     (effects (font (size 1 1) (thickness 0.15)))
@@
   (segment (start 181.365 109.719) (end 181.356 109.728) (width 0.25) (layer F.Cu) (net 19))
   (segment (start 181.365 104.745) (end 181.365 109.719) (width 0.25) (layer F.Cu) (net 19))
-  (segment (start 176.765858 114.808) (end 181.356 109.728) (width 0.25) (layer F.Cu) (net 19))
-  (segment (start 133.096 115.316) (end 176.765858 114.808) (width 0.25) (layer F.Cu) (net 19))
-  (segment (start 124.114999 105.758001) (end 133.096 115.316) (width 0.25) (layer F.Cu) (net 19))
-  (segment (start 124.114999 94.196591) (end 124.114999 105.758001) (width 0.25) (layer F.Cu) (net 19))
-  (segment (start 133.55559 84.756) (end 124.114999 94.196591) (width 0.25) (layer F.Cu) (net 19))
-  (segment (start 145.088 84.756) (end 143.314 84.756) (width 0.25) (layer F.Cu) (net 19))
+  (segment (start 132.338 84.756) (end 132.588 84.756) (width 0.25) (layer F.Cu) (net 19))
+  (segment (start 124.114999 92.979001) (end 132.338 84.756) (width 0.25) (layer F.Cu) (net 19))
+  (segment (start 181.356 109.728) (end 176.765858 114.808) (width 0.25) (layer F.Cu) (net 19))
+  (segment (start 133.096 115.316) (end 124.114999 105.758001) (width 0.25) (layer F.Cu) (net 19))
+  (segment (start 176.765858 114.808) (end 133.096 115.316) (width 0.25) (layer F.Cu) (net 19))
+  (segment (start 124.114999 105.758001) (end 124.114999 92.979001) (width 0.25) (layer F.Cu) (net 19))
   (segment (start 176.285 109.719) (end 176.276 109.728) (width 0.25) (layer F.Cu) (net 20))
   (segment (start 176.285 104.745) (end 176.285 109.719) (width 0.25) (layer F.Cu) (net 20))
